File: RhythmGamePicoBreakout/RhythmGamePicoBreakout.kicad_sch (KiCad schematic)
At the start: 65 parts, among them J1 BUTTON0, J10 BUTTON9, J11 BUTTON10, J12 QE1, J13 QE2, J14 Conn_01x02_Pin, J15 RGB1, J16 RGB2, J17 Conn_01x05, J18 USB_C_Receptacle_USB2.0, J19 Conn_01x05, J2 BUTTON1, J3 BUTTON2, J4 BUTTON3, J5 BUTTON4, J6 BUTTON5, J7 BUTTON6, J8 BUTTON7, J9 BUTTON8, Q1 LSI1012LT1G, Q10 LSI1012LT1G, Q11 LSI1012LT1G, Q12 LSI1012LT1G, Q13 LSI1012LT1G, Q2 LSI1012LT1G, Q3 LSI1012LT1G, Q4 LSI1012LT1G, Q5 LSI1012LT1G, Q6 LSI1012LT1G, Q7 LSI1012LT1G, Q8 LSI1012LT1G, Q9 LSI1012LT1G, SW1 SW_Push, SW2 SW_Push, U1 RP2040, U2 SRV05-4, U3 W25Q128JVS, U4 XC6206PxxxMR, Y1 Crystal_GND24

Commit message: Updated Schematics and PCB design
Parts:
- removed C3: 100n, Capacitor_SMD:C_0402_1005Metric_Pad0.74x0.62mm_HandSolder, symbol Device:C
- removed J19: Conn_01x05, Connector_PinSocket_2.00mm:PinSocket_1x05_P2.00mm_Vertical, symbol Connector_Generic:Conn_01x05
- removed Q12, Q13: LSI1012LT1G, Package_TO_SOT_SMD:SOT-23, symbol Transistor_FET:2N7000
- removed R9: 5.1K, Resistor_SMD:R_0402_1005Metric_Pad0.72x0.64mm_HandSolder, symbol Device:R
- removed SW2: SW_Push, Button_Switch_SMD:SW_SPST_REED_CT05-XXXX-G1, symbol Switch:SW_Push
- added C17: 0.33u, Capacitor_SMD:C_0402_1005Metric_Pad0.74x0.62mm_HandSolder, symbol Device:C
- added C18: 1u, Capacitor_SMD:C_0402_1005Metric_Pad0.74x0.62mm_HandSolder, symbol Device:C
- added C2: 100n, Capacitor_SMD:C_0402_1005Metric_Pad0.74x0.62mm_HandSolder, symbol Device:C
- added H1, H2, H3, H4: MountingHole, MountingHole:MountingHole_3.7mm, symbol Mechanical:MountingHole
- added J19: Conn_01x03, Connector_PinHeader_2.00mm:PinHeader_1x03_P2.00mm_Vertical, symbol Connector_Generic:Conn_01x03
- added J20: PS2 Header, Connector_JST:JST_XH_B8B-XH-AM_1x08_P2.50mm_Vertical, symbol Connector_Generic:Conn_01x08
- added J21: Conn_01x02_Pin, Connector_PinSocket_2.00mm:PinSocket_1x02_P2.00mm_Vertical, symbol Connector:Conn_01x02_Pin
- added U5: SN74HCT125D, SN74HCT125D:SOIC127P600X175-14N, symbol SN74HCT125D:SN74HCT125D
- added U6: LM7805_TO220, Package_TO_SOT_THT:TO-220-3_Vertical, symbol Regulator_Linear:LM7805_TO220
- C15, C16: value 22p -> 27p
- J15, J16: footprint Connector_JST:JST_XH_B4B-XH-AM_1x04_P2.50mm_Vertical -> Connector_JST:JST_XH_B3B-XH-AM_1x03_P2.50mm_Vertical
- J17: value Conn_01x05 -> USB Header
- R1, R2: value 22Ω -> 27Ω
- R7: value 1K -> 5.1K; now in the parts list
- R8: value 5.1K -> 1K
- RESET1: renamed from SW1; value SW_Push -> BOOTSEL; footprint Button_Switch_SMD:SW_SPST_REED_CT05-XXXX-G1 -> Button_Switch_SMD:SW_Push_1P1T_NO_CK_KSC6xxJ
- renumbered C2 to C13
Connections:
- net +1V1: now also C2.1, C4.1, C2.1
- net +3V3: now also R7.1, J20.6 (Pin_6); no longer R5.1, R8.1
- net +5V: now also J17.5 (Pin_5), C18.1, U6.3 (VO); no longer J17.1 (Pin_1)
- net BT0: now also U1.6 (GPIO4); no longer U1.2 (GPIO0)
- net BT1: now also U1.8 (GPIO6); no longer U1.3 (GPIO1)
- net BT10: now also U1.34 (GPIO22); no longer U1.13 (GPIO10)
- net BT2: now also U1.11 (GPIO8); no longer U1.4 (GPIO2)
- net BT3: now also U1.13 (GPIO10); no longer U1.5 (GPIO3)
- net BT4: now also U1.15 (GPIO12); no longer U1.6 (GPIO4)
- net BT5: now also U1.17 (GPIO14); no longer U1.7 (GPIO5)
- net BT6: now also U1.27 (GPIO16); no longer U1.8 (GPIO6)
- net BT7: now also U1.29 (GPIO18); no longer U1.9 (GPIO7)
- net BT8: now also U1.31 (GPIO20); no longer U1.11 (GPIO8)
- net BT9: now also U1.36 (GPIO24); no longer U1.12 (GPIO9)
- net GND: now also J17.1 (Pin_1), J17.2 (Pin_2), U1.19 (TESTEN), U1.57 (GND), C17.2, C18.2, C2.2, J19.2 (Pin_2), J20.1 (Pin_1), J21.2 (Pin_2), U5.1 (1~OE), U5.10 (3~OE), U5.13 (4~OE), U5.4 (2~OE), U5.7 (GND), U6.2 (GND); no longer J17.4 (Pin_4), J17.5 (Pin_5)
- net GP25: now also J14.1 (Pin_1), J20.5 (Pin_5); no longer J14.2 (Pin_2)
- net LED0: now also U1.5 (GPIO3); no longer U1.14 (GPIO11)
- net LED1: now also U1.7 (GPIO5); no longer U1.15 (GPIO12)
- net LED10: now also J20.7 (Pin_7)
- net LED2: now also U1.9 (GPIO7); no longer U1.16 (GPIO13)
- net LED3: now also U1.12 (GPIO9); no longer U1.17 (GPIO14)
- net LED4: now also U1.14 (GPIO11); no longer U1.18 (GPIO15)
- net LED5: now also U1.16 (GPIO13); no longer U1.27 (GPIO16)
- net LED6: now also U1.18 (GPIO15); no longer U1.28 (GPIO17)
- net LED7: now also U1.28 (GPIO17); no longer U1.29 (GPIO18)
- net LED9: now also U1.35 (GPIO23); no longer U1.31 (GPIO20)
- net QE1A: now also U1.3 (GPIO1); no longer U1.38 (GPIO26_ADC0)
- net QE1B: now also U1.2 (GPIO0); no longer U1.39 (GPIO27_ADC1)
- net Q_SEL: now also R5.2, R8.2; no longer R7.2
- net RGB1: now also J15.3 (Pin_3), U5.3 (1Y); no longer U1.34 (GPIO22)
- net RGB2: now also J16.3 (Pin_3), U5.6 (2Y); no longer U1.35 (GPIO23)
- net SWCLK: now also J19.1 (Pin_1)
- net SWD: now also J19.3 (Pin_3)
- net USB_DM: now also J17.4 (Pin_4), U2.4 (IO3); no longer J17.2 (Pin_2), U2.3 (IO2)
- net USB_DP: now also U2.3 (IO2); no longer U2.1 (IO1)
- net VBUS: now also U5.14 (VCC)
- net RUN: now reaches U1.26 (RUN)
- net RUN: now also J21.1 (Pin_1)
- removed net GP24: J14.1 (Pin_1), U1.36 (GPIO24)
- net QE2A renamed PS2CLK
- net PS2CLK: now also U1.41 (GPIO29_ADC3), J20.2 (Pin_2); no longer U1.40 (GPIO28_ADC2)
- net QE2B renamed PS2COMM
- net PS2COMM: now also U1.40 (GPIO28_ADC2), J20.3 (Pin_3); no longer U1.41 (GPIO29_ADC3)
- net RESET renamed USB_BOOT
- net USB_BOOT: now also R8.1; no longer R5.2
- new net: R5.1, R7.2
- new net GP26: J14.2 (Pin_2), J20.4 (Pin_4), U1.38 (GPIO26_ADC0)
- new net PS2_9V: C17.1, J20.8 (Pin_8), U6.1 (VI)
- new net RGBIn1: U1.4 (GPIO2), U5.2 (1A)
- new net RGBIn2: U1.39 (GPIO27_ADC1), U5.5 (2A)
- no-connect marks 4 -> 8
Other:
- note added: "PlayStation 2"
- note added: "Subject to change"
- moved on the sheet: C1, C10, C11, C12, C13, C14, C15, C16, C2, C4, C5, C6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

Commit message: Updated schematics and completely redone tracing
Parts:
- J19: value Conn_01x03 -> DEBUG
Connections:
- net BT0: now also U1.7 (GPIO5); no longer U1.6 (GPIO4)
- net BT1: now also U1.9 (GPIO7); no longer U1.8 (GPIO6)
- net BT2: now also U1.12 (GPIO9); no longer U1.11 (GPIO8)
- net BT3: now also U1.14 (GPIO11); no longer U1.13 (GPIO10)
- net BT4: now also U1.16 (GPIO13); no longer U1.15 (GPIO12)
- net BT5: now also U1.18 (GPIO15); no longer U1.17 (GPIO14)
- net BT6: now also U1.28 (GPIO17); no longer U1.27 (GPIO16)
- net BT7: now also U1.30 (GPIO19); no longer U1.29 (GPIO18)
- net BT8: now also U1.32 (GPIO21); no longer U1.31 (GPIO20)
- net GP25: now also U1.38 (GPIO26_ADC0); no longer U1.37 (GPIO25)
- net GP26: now also U1.39 (GPIO27_ADC1); no longer U1.38 (GPIO26_ADC0)
- net LED0: now also U1.6 (GPIO4); no longer U1.5 (GPIO3)
- net LED1: now also U1.8 (GPIO6); no longer U1.7 (GPIO5)
- net LED10: now also U1.35 (GPIO23); no longer U1.32 (GPIO21)
- net LED2: now also U1.11 (GPIO8); no longer U1.9 (GPIO7)
- net LED3: now also U1.13 (GPIO10); no longer U1.12 (GPIO9)
- net LED4: now also U1.15 (GPIO12); no longer U1.14 (GPIO11)
- net LED5: now also U1.17 (GPIO14); no longer U1.16 (GPIO13)
- net LED6: now also U1.27 (GPIO16); no longer U1.18 (GPIO15)
- net LED7: now also U1.29 (GPIO18); no longer U1.28 (GPIO17)
- net LED8: now also U1.31 (GPIO20); no longer U1.30 (GPIO19)
- net LED9: now also U1.37 (GPIO25); no longer U1.35 (GPIO23)
- net RGB1: now also U5.8 (3Y); no longer U5.3 (1Y)
- net RGB2: now also U5.11 (4Y); no longer U5.6 (2Y)
- net RGBIn1: now also U1.5 (GPIO3), U5.9 (3A); no longer U1.4 (GPIO2), U5.2 (1A)
- net RGBIn2: now also U1.4 (GPIO2), U5.12 (4A); no longer U1.39 (GPIO27_ADC1), U5.5 (2A)
- net USB_DM: now also U2.1 (IO1); no longer U2.4 (IO3)
- net USB_DP: now also U2.6 (IO4); no longer U2.3 (IO2)
