File: Axion-Board.kicad_pcb (KiCad board)
At the start: 2 copper layers, 84 x 54.5 mm, 78 parts, among them J1 USB_C_Receptacle_USB2.0, J14 QE2B, J15 RGB2, J16 RGB1, J17 QE1, J18 QE2, J19 USB Header, J2 SWD, J20 PS2 Header, J21 QE2A, J3 QE1A, J4 QE1B, J6 GPIO, J7 GPIO, Q1 BSS138, Q10 BSS138, Q11 BSS138, Q2 BSS138, Q3 BSS138, Q4 BSS138, Q5 BSS138, Q6 BSS138, Q7 BSS138, Q8 BSS138, Q9 BSS138, SW1 SW_Push, U1 W25Q128JVS, U2 USBLC6-2SC6, U3 RP2040, U4 XC6206PxxxMR-Regulator_Linear, U5 SN74HCT125DR, U6 78M05_TO252-3, Y1 12MHz

Commit message: Fixed the mosfet wiring
Parts:
- BTN1: value BUTTON7 -> BUTTON1
- BTN2: value BUTTON6 -> BUTTON2
- BTN3: value BUTTON5 -> BUTTON3
- BTN5: value BUTTON3 -> BUTTON5
- BTN6: value BUTTON2 -> BUTTON6
- BTN7: value BUTTON1 -> BUTTON7
- BTN8: value BUTTON0 -> BUTTON8
- C2, C3: value 22pF -> 15pF
- moved Q7 46.4 mm to (124.4, 61.2), turned to 180 degrees
- moved Q11 38.9 mm to (120.4, 90.4), turned to 90 degrees
- moved Q10 37.3 mm to (133.8, 89.2), turned to 90 degrees
- moved Q9 35.6 mm to (147.3, 88.6), turned to 90 degrees
- moved Q6 26.1 mm to (148.3, 63.1), turned to 90 degrees
- moved Q5 23.9 mm to (170.8, 93.6), turned to 90 degrees
- moved Q4 21.4 mm to (156.0, 89.0), turned to 90 degrees
- moved Q2 14.0 mm to (143.1, 88.3), turned to 90 degrees
- moved Q1 8.56 mm to (129.1, 88.9), turned to 90 degrees
- moved Q8 5.03 mm to (160.8, 90.3), turned to 90 degrees
- moved Q3 0.96 mm to (113.5, 89.0), turned to 90 degrees
Connections:
- Q1 pad 1: /LED7 -> /LED6
- Q1 pad 2: Net-(BTN7-Pin_2) -> GND
- Q1 pad 3: GND -> Net-(BTN6-Pin_2)
- Q10 pad 1: /LED0 -> /LED5
- Q10 pad 2: Net-(BTN0-Pin_2) -> GND
- Q10 pad 3: GND -> Net-(BTN5-Pin_2)
- Q11 pad 1: /LED9 -> /LED7
- Q11 pad 2: Net-(BTN9-Pin_2) -> GND
- Q11 pad 3: GND -> Net-(BTN7-Pin_2)
- Q2 pad 1: /LED6 -> /LED4
- Q2 pad 2: Net-(BTN6-Pin_2) -> GND
- Q2 pad 3: GND -> Net-(BTN4-Pin_2)
- Q3 pad 2: Net-(BTN8-Pin_2) -> GND
- Q3 pad 3: GND -> Net-(BTN8-Pin_2)
- Q4 pad 1: /LED5 -> /LED2
- Q4 pad 2: Net-(BTN5-Pin_2) -> GND
- Q4 pad 3: GND -> Net-(BTN2-Pin_2)
- Q5 pad 1: /LED3 -> /LED0
- Q5 pad 2: Net-(BTN3-Pin_2) -> GND
- Q5 pad 3: GND -> Net-(BTN0-Pin_2)
- Q6 pad 1: /LED4 -> /LED9
- Q6 pad 2: Net-(BTN4-Pin_2) -> GND
- Q6 pad 3: GND -> Net-(BTN9-Pin_2)
- Q7 pad 1: /LED1 -> /LED10
- Q7 pad 2: Net-(BTN1-Pin_2) -> GND
- Q7 pad 3: GND -> Net-(BTN10-Pin_2)
- Q8 pad 1: /LED2 -> /LED1
- Q8 pad 2: Net-(BTN2-Pin_2) -> GND
- Q8 pad 3: GND -> Net-(BTN1-Pin_2)
- Q9 pad 1: /LED10 -> /LED3
- Q9 pad 2: Net-(BTN10-Pin_2) -> GND
- Q9 pad 3: GND -> Net-(BTN3-Pin_2)
Routing:
- net VBUS: track 135.9 -> 146.9 mm, vias 12 -> 9
- net GND: track 221.8 -> 231.1 mm, vias 61 -> 63
- net +3V3: track 82.6 -> 86.5 mm, vias 6 -> 7
- net /LED7: track 23.3 -> 26.9 mm
- net /LED5: track 11.8 -> 15.3 mm
- net /LED1: track 30.7 -> 34.1 mm
- net /LED8: track 28.8 -> 32.0 mm
- net Net-(BTN0-Pin_2): track 8.65 -> 11.3 mm
- net /LED6: track 15.6 -> 17.9 mm
- net Net-(BTN4-Pin_2): track 13.7 -> 15.9 mm
- net Net-(BTN6-Pin_2): track 13.5 -> 15.6 mm
- net Net-(BTN2-Pin_2): track 13.4 -> 15.4 mm
- net /LED4: track 7.29 -> 9.24 mm
- net /LED3: track 10.5 -> 12.2 mm
- net Net-(BTN8-Pin_2): track 13.1 -> 14.7 mm
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Other:
- board text removed: "3d model loli ice cream drip video"
- board text removed: "holy shit this is so fucking aesome. Each navigator costs like 30-50 dollars to unlock but godamn im almost buckling"
- board text removed: "seeing sehun replied to a link of mine with {dblquote}holy shit this is sofucking awesome{dblquote} and hoping he played my bms and liked it before it sinks in that he was replying to the fucking sdvx"

Commit message: Added turntable LED header
Parts:
- added LED: LED, Connector_JST:JST_XH_B2B-XH-A_1x02_P2.50mm_Vertical, F.Cu at (103.3, 86.8)
- moved R8 0.37 mm to (108.7, 76.5)
- moved J16 0.31 mm to (103.4, 79.9)
Connections:
- net /GP18 renamed /GP20
- net /GP19 renamed /GP21
Routing:
- net GND: track 231.1 -> 240.1 mm
- net VBUS: track 146.9 -> 148.9 mm, vias 9 -> 11
Other:
- board text added: "GP21 GP20"
- board text added: "[G|V]"
- board text removed: "GP19 GP18"
